Commit message: sensor success test

File: src/rmitbot_cliff_sensor/urdf/cliff_sensor.xacro (robot description, xacro)
@@ -14,17 +14,4 @@
         <!-- Cliff sensor link (visual representation) -->
         <link name="${name}_link">
-            <visual>
-                <geometry>
-                    <box size="0.02 0.02 0.01"/>
-                </geometry>
-                <material name="black">
-                    <color rgba="0.1 0.1 0.1 1"/>
-                </material>
-            </visual>
-            <collision>
-                <geometry>
-                    <box size="0.02 0.02 0.01"/>
-                </geometry>
-            </collision>
             <inertial>
                 <mass value="0.01"/>
@@ -42,5 +29,5 @@
                 <topic>sensors/cliff/${name}</topic>
                 <gz_frame_id>${name}_link</gz_frame_id>
-                <ray>
+                <lidar>
                     <scan>
                         <horizontal>
@@ -51,12 +38,12 @@
                         </horizontal>
                         <vertical>
-                            <samples>1</samples>
+                            <samples>3</samples>
                             <resolution>1</resolution>
-                            <min_angle>0.0</min_angle>
-                            <max_angle>0.0</max_angle>
+                            <min_angle>-0.01</min_angle>
+                            <max_angle>0.01</max_angle>
                         </vertical>
                     </scan>
                     <range>
-                        <min>0.01</min>
+                        <min>0.001</min>
                         <max>1.5</max>
                         <resolution>0.005</resolution>
@@ -67,5 +54,5 @@
                         <stddev>0.005</stddev>
                     </noise>
-                </ray>
+                </lidar>
             </sensor>
             <visual>

File: src/rmitbot_description/urdf/rmitbot.urdf.xacro (robot description, xacro)
@@ -2,4 +2,5 @@
 <robot name="rmitbot"
     xmlns:xacro="http://ros.org/wiki/xacro">
+    <xacro:arg name="use_sim" default="true"/>
     <xacro:include filename="$(find rmitbot_description)/urdf/rmitbot_platform.xacro" />
     <xacro:include filename="$(find rmitbot_description)/urdf/rmitbot_gazebo.xacro" />
@@ -11,9 +12,9 @@
     <!-- Front Left Cliff Sensor (Floating on top-left corner, pointing straight down) -->
     <xacro:cliff_sensor name="cliff_fl" parent="base_link">
-        <origin xyz="0.14 0.17 0.12" rpy="0 1.5708 0" />
+        <origin xyz="0.16 0.24 0.11" rpy="0 1.5708 0" />
     </xacro:cliff_sensor>
     <!-- Front Right Cliff Sensor (Floating on top-right corner, pointing straight down) -->
     <xacro:cliff_sensor name="cliff_fr" parent="base_link">
-        <origin xyz="0.14 -0.17 0.12" rpy="0 1.5708 0" />
+        <origin xyz="0.16 -0.24 0.11" rpy="0 1.5708 0" />
     </xacro:cliff_sensor>
 </robot>

File: src/rmitbot_description/urdf/rmitbot_ros2_control.xacro (robot description, xacro)
@@ -2,9 +2,16 @@
 <robot name="rmitbot" xmlns:xacro="http://www.ros.org/wiki/xacro" >
     <ros2_control name="RobotSystem" type="system">
-        <hardware>
-            <plugin>rmitbot_firmware/RmitbotInterface</plugin>
-            <!-- <param name="port">/dev/esp32</param> -->
-            <param name="port">/dev/ttyUSB0</param>
-        </hardware>
+        <xacro:if value="$(arg use_sim)">
+            <hardware>
+                <plugin>gz_ros2_control/GazeboSimSystem</plugin>
+            </hardware>
+        </xacro:if>
+        <xacro:unless value="$(arg use_sim)">
+            <hardware>
+                <plugin>rmitbot_firmware/RmitbotInterface</plugin>
+                <!-- <param name="port">/dev/esp32</param> -->
+                <param name="port">/dev/ttyUSB0</param>
+            </hardware>
+        </xacro:unless>
         <joint name="front_left_wheel_joint">
             <command_interface name="velocity">

Commit message: sensor success test

File: src/rmitbot_cliff_sensor/urdf/cliff_sensor.xacro (robot description, xacro)
@@ -14,4 +14,12 @@
         <!-- Cliff sensor link (visual representation) -->
         <link name="${name}_link">
+            <visual>
+                <geometry>
+                    <box size="0.02 0.02 0.01"/>
+                </geometry>
+                <material name="black">
+                    <color rgba="0.1 0.1 0.1 1"/>
+                </material>
+            </visual>
             <inertial>
                 <mass value="0.01"/>
