Commit message: sim push

File: TEMP/lesson5_ws/src/rmitbot_description/urdf/rmitbot.urdf.xacro (robot description, xacro)
@@ -5,4 +5,5 @@
 <robot name="rmitbot"
     xmlns:xacro="http://ros.org/wiki/xacro">
+    <xacro:arg name="prefix" default=""/>
     <xacro:include filename="$(find rmitbot_description)/urdf/rmitbot_platform.xacro" />
     <xacro:include filename="$(find rmitbot_description)/urdf/rmitbot_gazebo.xacro" />
@@ -10,3 +11,8 @@
     <xacro:include filename="$(find rmitbot_description)/urdf/rmitbot_imu.xacro" />
     <xacro:include filename="$(find rmitbot_description)/urdf/rmitbot_laser.xacro" />
+    <xacro:rmitbot_platform prefix="$(arg prefix)"/>
+<xacro:rmitbot_gazebo prefix="$(arg prefix)"/>
+<xacro:rmitbot_ros2_control prefix="$(arg prefix)"/>
+<xacro:rmitbot_imu prefix="$(arg prefix)"/>
+<xacro:rmitbot_laser prefix="$(arg prefix)"/>
 </robot>

File: TEMP/lesson5_ws/src/rmitbot_description/urdf/rmitbot_gazebo.xacro (robot description, xacro)
@@ -2,8 +2,9 @@
 <!-- Gazebo file contains information regarding the lnks's physics (e.g., friction, stiffness, damping) -->
 <robot name="rmitbot" xmlns:xacro="http://ros.org/wiki/xacro" xmlns:gz="http://gazebosim.org/schema">
+<xacro:macro name="rmitbot_gazebo" params="prefix">
   <!-- Wheels -->
      <!-- To emulate Mecanum wheels in Gazebo with spherical collisions it
   requires a custom friction model so the vehicle can strafe left to right -->
-  <gazebo reference='front_left_wheel'>
+  <gazebo reference='${prefix}front_left_wheel'>
     <collision>
       <surface>
@@ -12,6 +13,6 @@
             <mu>1.0</mu>
             <mu2>0.0</mu2>
-            <!-- <fdir1 gz:expressed_in="base_link">1 -1 0</fdir1> -->
-            <fdir1 gz:expressed_in="base_footprint">1 -1 0</fdir1>
+            <!-- <fdir1 gz:expressed_in="${prefix}base_link">1 -1 0</fdir1> -->
+            <fdir1 gz:expressed_in="${prefix}base_footprint">1 -1 0</fdir1>
           </ode>
         </friction>
@@ -19,5 +20,5 @@
     </collision>
   </gazebo>
-  <gazebo reference='front_right_wheel'>
+  <gazebo reference='${prefix}front_right_wheel'>
     <collision>
       <surface>
@@ -26,6 +27,6 @@
             <mu>1.0</mu>
             <mu2>0.0</mu2>
-            <!-- <fdir1 gz:expressed_in="base_link">1 1 0</fdir1> -->
-            <fdir1 gz:expressed_in="base_footprint">1 1 0</fdir1>
+            <!-- <fdir1 gz:expressed_in="${prefix}base_link">1 1 0</fdir1> -->
+            <fdir1 gz:expressed_in="${prefix}base_footprint">1 1 0</fdir1>
           </ode>
         </friction>
@@ -33,5 +34,5 @@
     </collision>
   </gazebo>
-  <gazebo reference='rear_left_wheel'>
+  <gazebo reference='${prefix}rear_left_wheel'>
     <collision>
       <surface>
@@ -40,6 +41,6 @@
             <mu>1.0</mu>
             <mu2>0.0</mu2>
-            <!-- <fdir1 gz:expressed_in="base_link">1 1 0</fdir1> -->
-            <fdir1 gz:expressed_in="base_footprint">1 1 0</fdir1>
+            <!-- <fdir1 gz:expressed_in="${prefix}base_link">1 1 0</fdir1> -->
+            <fdir1 gz:expressed_in="${prefix}base_footprint">1 1 0</fdir1>
           </ode>
         </friction>
@@ -47,5 +48,5 @@
     </collision>
   </gazebo>
-  <gazebo reference='rear_right_wheel'>
+  <gazebo reference='${prefix}rear_right_wheel'>
     <collision>
       <surface>
@@ -54,6 +55,6 @@
             <mu>1.0</mu>
             <mu2>0.0</mu2>
-            <!-- <fdir1 gz:expressed_in="base_link">1 -1 0</fdir1> -->
-            <fdir1 gz:expressed_in="base_footprint">1 -1 0</fdir1>
+            <!-- <fdir1 gz:expressed_in="${prefix}base_link">1 -1 0</fdir1> -->
+            <fdir1 gz:expressed_in="${prefix}base_footprint">1 -1 0</fdir1>
           </ode>
         </friction>
@@ -61,3 +62,4 @@
     </collision>
   </gazebo>
+  </xacro:macro>
 </robot>

File: TEMP/lesson5_ws/src/rmitbot_description/urdf/rmitbot_imu.xacro (robot description, xacro)
@@ -1,5 +1,6 @@
 <?xml version="1.0"?>
 <robot xmlns:xacro="http://www.ros.org/wiki/xacro" name="rmitbot">
-    <link name="imu_link">
+<xacro:macro name="rmitbot_imu" params="prefix">
+    <link name="${prefix}imu_link">
         <inertial>
             <origin xyz="-0.0055 0.00017 0.00051" rpy="0 0 0" />
@@ -24,8 +25,8 @@
         </collision>
     </link>
-    <joint name="imu_joint" type="fixed">
+    <joint name="${prefix}imu_joint" type="fixed">
         <origin xyz="0 0 0.1" rpy="0 0 0" />
-        <parent link="base_link" />
-        <child link="imu_link" />
+        <parent link="${prefix}base_link" />
+        <child link="${prefix}imu_link" />
         <axis xyz="0 0 0" />
     </joint>
@@ -36,10 +37,10 @@
     </gazebo>
     <!-- Gazebo parameters for IMU, with noise-->
-  <gazebo reference="imu_link">
-    <sensor name="imu" type="imu">
+  <gazebo reference="${prefix}imu_link">
+    <sensor name="${prefix}imu" type="imu">
       <always_on>true</always_on>
       <update_rate>100</update_rate>
-      <gz_frame_id>imu_link</gz_frame_id>
-      <topic>imu</topic>
+      <gz_frame_id>${prefix}imu_link</gz_frame_id>
+      <topic>${prefix[:-1]}_imu</topic>
       <imu>
         <angular_velocity>
@@ -86,3 +87,4 @@
     </sensor>
   </gazebo>
+</xacro:macro>
 </robot>

File: TEMP/lesson5_ws/src/rmitbot_description/urdf/rmitbot_laser.xacro (robot description, xacro)
@@ -1,5 +1,6 @@
 <?xml version="1.0"?>
-<robot xmlns:xacro="http://www.ros.org/wiki/xacro" name="rmitbot">
-    <link name="laser_link">
+<robot xmlns:xacro="http://www.ros.org/wiki/xacro">
+ <xacro:macro name="rmitbot_laser" params="prefix">
+    <link name="${prefix}laser_link">
         <inertial>
             <origin xyz="-0.012 -0.00038 -0.017" rpy="0 0 0" />
@@ -21,21 +22,21 @@
         </collision>
     </link>
-    <joint name="laser_joint" type="fixed">
+    <joint name="${prefix}laser_joint" type="fixed">
         <origin xyz="0. 0. 0.14" rpy="0 0 0" />
-        <parent link="base_link" />
-        <child link="laser_link" />
+        <parent link="${prefix}base_link" />
+        <child link="${prefix}laser_link" />
         <axis xyz="0 0 0" />
     </joint>
-    <gazebo reference="laser_link">
-        <sensor name="lidar" type="gpu_lidar">
-            <!-- <sensor name="lidar" type="ray"> -->
-            <plugin filename="gz-sim-sensors-system" name="gz::sim::systems::Sensors">
+    <gazebo reference="${prefix}laser_link">
+        <!-- <sensor name="${prefix}lidar" type="gpu_lidar"> -->
+            <sensor name="${prefix}lidar" type="gpu_lidar">
+            <!-- <plugin filename="gz-sim-sensors-system" name="gz::sim::systems::Sensors">
                 <render_engine>ogre</render_engine>
-            </plugin>
+            </plugin> -->
             <always_on>true</always_on>
             <visualize>true</visualize>
-            <topic>scan</topic>
+            <topic>${prefix[:-1]}_scan</topic>
             <update_rate>5</update_rate>
-            <gz_frame_id>laser_link</gz_frame_id>
+            <gz_frame_id>${prefix}laser_link</gz_frame_id>
             <lidar>
                 <!-- <ray> -->
@@ -68,3 +69,4 @@
         </sensor>
     </gazebo>
+    </xacro:macro>
 </robot>

File: TEMP/lesson5_ws/src/rmitbot_description/urdf/rmitbot_platform.xacro (robot description, xacro)
@@ -1,4 +1,4 @@
 <?xml version="1.0"?>
-<robot name="rmitbot" xmlns:xacro="http://www.ros.org/wiki/xacro" xmlns:gz="http://gazebosim.org/schema">
+<robot xmlns:xacro="http://www.ros.org/wiki/xacro" xmlns:gz="http://gazebosim.org/schema">
   <material name="orange">
     <color rgba="0.8 0.4 0.0 1.0" />
@@ -10,12 +10,13 @@
     <color rgba="1 1 1 1.0" />
   </material>
-  <link name="base_footprint" />
-  <joint name="base_joint" type="fixed">
-    <parent link="base_footprint" />
-    <child link="base_link" />
+<xacro:macro name="rmitbot_platform" params="prefix">
+  <link name="${prefix}base_footprint" />
+  <joint name="${prefix}base_joint" type="fixed">
+    <parent link="${prefix}base_footprint" />
+    <child link="${prefix}base_link" />
     <origin xyz="0 0 0.05" rpy="0 0 0" />
   </joint>
   <!-- Base Link -->
-  <link name="base_link">
+  <link name="${prefix}base_link">
     <collision>
       <origin xyz="0 0 0.05" rpy="0 0 0" />
@@ -44,12 +45,12 @@
   </link>
   <!-- front left wheel -->
-  <joint name="front_left_wheel_joint" type="continuous">
+  <joint name="${prefix}front_left_wheel_joint" type="continuous">
     <origin xyz="0.14 0.15 0" rpy="-${pi/2} 0 0" />
-    <parent link="base_link" />
-    <child link="front_left_wheel" />
+    <parent link="${prefix}base_link" />
+    <child link="${prefix}front_left_wheel" />
     <axis xyz="0 0 1" />
     <dynamics damping="0.2" />
   </joint>
-  <link name="front_left_wheel">
+  <link name="${prefix}front_left_wheel">
     <collision>
       <!-- <origin xyz="0 0 .06" rpy="0 0 0" /> -->
@@ -81,12 +82,12 @@
   </link>
   <!-- front right wheel -->
-  <joint name="front_right_wheel_joint" type="continuous">
+  <joint name="${prefix}front_right_wheel_joint" type="continuous">
     <origin xyz="0.14 -0.15 0." rpy="-${pi/2} 0 0" />
-    <parent link="base_link" />
-    <child link="front_right_wheel" />
+    <parent link="${prefix}base_link" />
+    <child link="${prefix}front_right_wheel" />
     <axis xyz="0 0 1" />
     <dynamics damping="0.2" />
   </joint>
-  <link name="front_right_wheel">
+  <link name="${prefix}front_right_wheel">
     <collision>
       <!-- <origin xyz="0 0 -.06" rpy="0 0 0" /> -->
@@ -116,12 +117,12 @@
   </link>
   <!-- rear left wheel -->
-  <joint name="rear_left_wheel_joint" type="continuous">
+  <joint name="${prefix}rear_left_wheel_joint" type="continuous">
     <origin xyz="-0.14 0.15 0." rpy="-${pi/2} 0 0" />
-    <parent link="base_link" />
-    <child link="rear_left_wheel" />
+    <parent link="${prefix}base_link" />
+    <child link="${prefix}rear_left_wheel" />
     <axis xyz="0 0 1" />
     <dynamics damping="0.2" />
   </joint>
-  <link name="rear_left_wheel">
+  <link name="${prefix}rear_left_wheel">
     <collision>
       <!-- <origin xyz="0 0 .06" rpy="0 0 0" /> -->
@@ -152,12 +153,12 @@
   </link>
   <!-- rear right wheel -->
-  <joint name="rear_right_wheel_joint" type="continuous">
+  <joint name="${prefix}rear_right_wheel_joint" type="continuous">
     <origin xyz="-0.14 -0.15 0." rpy="-${pi/2} 0 0" />
-    <parent link="base_link" />
-    <child link="rear_right_wheel" />
+    <parent link="${prefix}base_link" />
+    <child link="${prefix}rear_right_wheel" />
     <axis xyz="0 0 1" />
     <dynamics damping="0.2" />
   </joint>
-  <link name="rear_right_wheel">
+  <link name="${prefix}rear_right_wheel">
     <collision>
       <!-- <origin xyz="0 0 -.06" rpy="0 0 0" /> -->
@@ -187,3 +188,4 @@
     </inertial>
   </link>
+  </xacro:macro>
 </robot>

File: TEMP/lesson5_ws/src/rmitbot_description/urdf/rmitbot_ros2_control.xacro (robot description, xacro)
@@ -1,9 +1,12 @@
 <?xml version="1.0"?>
-<robot name="rmitbot" xmlns:xacro="http://www.ros.org/wiki/xacro"> Define the vehicles hardware,
-    command and state interfaces <ros2_control name="GazeboSimSystem" type="system">
+<robot name="rmitbot" xmlns:xacro="http://www.ros.org/wiki/xacro">
+<!-- Define the vehicles hardware,
+    command and state interfaces  -->
+     <xacro:macro name="rmitbot_ros2_control" params="prefix">
+     <ros2_control name="GazeboSimSystem" type="system">
         <hardware>
             <plugin>gz_ros2_control/GazeboSimSystem</plugin>
         </hardware>
-        <joint name="front_left_wheel_joint">
+        <joint name="${prefix}front_left_wheel_joint">
             <command_interface name="velocity">
                 <param name="min">-1</param>
@@ -13,5 +16,5 @@
             <state_interface name="velocity" />
         </joint>
-        <joint name="front_right_wheel_joint">
+        <joint name="${prefix}front_right_wheel_joint">
             <command_interface name="velocity">
                 <param name="min">-1</param>
@@ -21,5 +24,5 @@
             <state_interface name="velocity" />
         </joint>
-        <joint name="rear_left_wheel_joint">
+        <joint name="${prefix}rear_left_wheel_joint">
             <command_interface name="velocity">
                 <param name="min">-1</param>
@@ -29,5 +32,5 @@
             <state_interface name="velocity" />
         </joint>
-        <joint name="rear_right_wheel_joint">
+        <joint name="${prefix}rear_right_wheel_joint">
             <command_interface name="velocity">
                 <param name="min">-1</param>
@@ -42,8 +45,10 @@
         <plugin filename="gz_ros2_control-system" name="gz_ros2_control::GazeboSimROS2ControlPlugin">
             <parameters>$(find rmitbot_controller)/config/rmitbot_controller.yaml</parameters>
-            <!-- <ros>
-                <remapping>/mecanum_drive_controller/odom:=/odom</remapping>
-            </ros> -->
+            <ros>
+                <namespace>${prefix[:-1]}</namespace>
+                <remapping>diff_drive_controller/odom:=/${prefix}odom</remapping>
+            </ros>
         </plugin>
     </gazebo>
+     </xacro:macro>
 </robot>
