Commit message: cliff test

File: src/rmitbot_description/urdf/rmitbot.urdf.xacro (robot description, xacro)
@@ -7,3 +7,13 @@
     <xacro:include filename="$(find rmitbot_description)/urdf/rmitbot_imu.xacro" />
     <xacro:include filename="$(find rmitbot_description)/urdf/rmitbot_laser.xacro" />
+    <!-- Include the cliff sensor macro -->
+    <xacro:include filename="$(find rmitbot_cliff_sensor)/urdf/cliff_sensor.xacro" />
+    <!-- Front Left Cliff Sensor (Floating on top-left corner, pointing straight down) -->
+    <xacro:cliff_sensor name="cliff_fl" parent="base_link">
+        <origin xyz="0.14 0.17 0.12" rpy="0 1.5708 0" />
+    </xacro:cliff_sensor>
+    <!-- Front Right Cliff Sensor (Floating on top-right corner, pointing straight down) -->
+    <xacro:cliff_sensor name="cliff_fr" parent="base_link">
+        <origin xyz="0.14 -0.17 0.12" rpy="0 1.5708 0" />
+    </xacro:cliff_sensor>
 </robot>

Commit message: Add all 6 cliff sensors to URDF and increase threshold

File: src/rmitbot_description/urdf/rmitbot.urdf.xacro (robot description, xacro)
@@ -10,11 +10,27 @@
     <!-- Include the cliff sensor macro -->
     <xacro:include filename="$(find rmitbot_cliff_sensor)/urdf/cliff_sensor.xacro" />
-    <!-- Front Left Cliff Sensor (Floating on top-left corner, pointing straight down) -->
-    <xacro:cliff_sensor name="cliff_fl" parent="base_link">
+    <!-- Cliff Sensor 0 (Front Center) -->
+    <xacro:cliff_sensor name="cliff_sensor_0" parent="base_link">
+        <origin xyz="0.2 0.0 0.11" rpy="0 1.5708 0" />
+    </xacro:cliff_sensor>
+    <!-- Cliff Sensor 1 (Front Right) -->
+    <xacro:cliff_sensor name="cliff_sensor_1" parent="base_link">
+        <origin xyz="0.16 -0.24 0.11" rpy="0 1.5708 0" />
+    </xacro:cliff_sensor>
+    <!-- Cliff Sensor 2 (Back Right) -->
+    <xacro:cliff_sensor name="cliff_sensor_2" parent="base_link">
+        <origin xyz="-0.16 -0.24 0.11" rpy="0 1.5708 0" />
+    </xacro:cliff_sensor>
+    <!-- Cliff Sensor 3 (Back Center) -->
+    <xacro:cliff_sensor name="cliff_sensor_3" parent="base_link">
+        <origin xyz="-0.2 0.0 0.11" rpy="0 1.5708 0" />
+    </xacro:cliff_sensor>
+    <!-- Cliff Sensor 4 (Back Left) -->
+    <xacro:cliff_sensor name="cliff_sensor_4" parent="base_link">
+        <origin xyz="-0.16 0.24 0.11" rpy="0 1.5708 0" />
+    </xacro:cliff_sensor>
+    <!-- Cliff Sensor 5 (Front Left) -->
+    <xacro:cliff_sensor name="cliff_sensor_5" parent="base_link">
         <origin xyz="0.16 0.24 0.11" rpy="0 1.5708 0" />
     </xacro:cliff_sensor>
-    <!-- Front Right Cliff Sensor (Floating on top-right corner, pointing straight down) -->
-    <xacro:cliff_sensor name="cliff_fr" parent="base_link">
-        <origin xyz="0.16 -0.24 0.11" rpy="0 1.5708 0" />
-    </xacro:cliff_sensor>
 </robot>

Commit message: Swarm deployment on physical hardware

File: src/rmitbot_description/urdf/rmitbot.urdf.xacro (robot description, xacro)
@@ -3,4 +3,5 @@
     xmlns:xacro="http://ros.org/wiki/xacro">
     <xacro:arg name="use_sim" default="false"/>
+    <xacro:arg name="prefix" default=""/>
     <xacro:include filename="$(find rmitbot_description)/urdf/rmitbot_platform.xacro" />
     <xacro:include filename="$(find rmitbot_description)/urdf/rmitbot_gazebo.xacro" />
@@ -8,4 +9,9 @@
     <xacro:include filename="$(find rmitbot_description)/urdf/rmitbot_imu.xacro" />
     <xacro:include filename="$(find rmitbot_description)/urdf/rmitbot_laser.xacro" />
+    <xacro:rmitbot_platform prefix="$(arg prefix)"/>
+    <xacro:rmitbot_gazebo prefix="$(arg prefix)"/>
+    <xacro:rmitbot_ros2_control prefix="$(arg prefix)"/>
+    <xacro:rmitbot_imu prefix="$(arg prefix)"/>
+    <xacro:rmitbot_laser prefix="$(arg prefix)"/>
     <!-- === CLIFF SENSORS DISABLED FOR BIG BOT ===
     <xacro:include filename="$(find rmitbot_cliff_sensor)/urdf/cliff_sensor.xacro" />

File: src/rmitbot_description/urdf/rmitbot_laser.xacro (robot description, xacro)
@@ -1,5 +1,6 @@
 <?xml version="1.0"?>
-<robot xmlns:xacro="http://www.ros.org/wiki/xacro" name="rmitbot">
-    <link name="laser_link">
+<robot xmlns:xacro="http://www.ros.org/wiki/xacro">
+ <xacro:macro name="rmitbot_laser" params="prefix">
+    <link name="${prefix}laser_link">
         <inertial>
             <origin xyz="-0.012 -0.00038 -0.017" rpy="0 0 0" />
@@ -21,22 +22,23 @@
         </collision>
     </link>
-    <joint name="laser_joint" type="fixed">
-        <!-- <origin xyz="0. 0. 0.12" rpy="0 0 3.14" /> -->
-        <origin xyz="0. 0. 0.12" rpy="0 0 0" />
-        <parent link="base_link" />
-        <child link="laser_link" />
+    <joint name="${prefix}laser_joint" type="fixed">
+        <origin xyz="0. 0. 0.14" rpy="0 0 0" />
+        <parent link="${prefix}base_link" />
+        <child link="${prefix}laser_link" />
         <axis xyz="0 0 0" />
     </joint>
-    <gazebo reference="laser_link">
-        <sensor name="lidar" type="gpu_lidar">
-            <plugin filename="gz-sim-sensors-system" name="gz::sim::systems::Sensors">
+    <gazebo reference="${prefix}laser_link">
+        <!-- <sensor name="${prefix}lidar" type="gpu_lidar"> -->
+            <sensor name="${prefix}lidar" type="gpu_lidar">
+            <!-- <plugin filename="gz-sim-sensors-system" name="gz::sim::systems::Sensors">
                 <render_engine>ogre</render_engine>
-            </plugin>
+            </plugin> -->
             <always_on>true</always_on>
             <visualize>true</visualize>
-            <topic>scan</topic>
+            <topic>${prefix[:-1]}_scan</topic>
             <update_rate>5</update_rate>
-            <gz_frame_id>laser_link</gz_frame_id>
+            <gz_frame_id>${prefix}laser_link</gz_frame_id>
             <lidar>
+                <!-- <ray> -->
                 <scan>
                     <horizontal>
@@ -46,4 +48,5 @@
                         <max_angle>6.280000</max_angle>
                     </horizontal>
+                    <!-- Dirty hack for fake lidar detections with ogre 1 rendering in VM -->
                     <vertical>
                         <samples>3</samples>
@@ -63,5 +66,7 @@
                 </noise>
             </lidar>
+            <!-- </ray> -->
         </sensor>
     </gazebo>
+    </xacro:macro>
 </robot>

File: src/rmitbot_description/urdf/rmitbot_platform.xacro (robot description, xacro)
@@ -1,4 +1,4 @@
 <?xml version="1.0"?>
-<robot name="rmitbot" xmlns:xacro="http://www.ros.org/wiki/xacro" xmlns:gz="http://gazebosim.org/schema">
+<robot xmlns:xacro="http://www.ros.org/wiki/xacro" xmlns:gz="http://gazebosim.org/schema">
   <material name="orange">
     <color rgba="0.8 0.4 0.0 1.0" />
@@ -10,11 +10,13 @@
     <color rgba="1 1 1 1.0" />
   </material>
-  <link name="base_footprint" />
-  <joint name="base_joint" type="fixed">
-    <parent link="base_footprint" />
-    <child link="base_link" />
+<xacro:macro name="rmitbot_platform" params="prefix">
+  <link name="${prefix}base_footprint" />
+  <joint name="${prefix}base_joint" type="fixed">
+    <parent link="${prefix}base_footprint" />
+    <child link="${prefix}base_link" />
     <origin xyz="0 0 0.05" rpy="0 0 0" />
   </joint>
-  <link name="base_link">
+  <!-- Base Link -->
+  <link name="${prefix}base_link">
     <collision>
       <origin xyz="0 0 0.05" rpy="0 0 0" />
@@ -42,13 +44,15 @@
     </inertial>
   </link>
-  <joint name="front_left_wheel_joint" type="continuous">
+  <!-- front left wheel -->
+  <joint name="${prefix}front_left_wheel_joint" type="continuous">
     <origin xyz="0.14 0.15 0" rpy="-${pi/2} 0 0" />
-    <parent link="base_link" />
-    <child link="front_left_wheel" />
+    <parent link="${prefix}base_link" />
+    <child link="${prefix}front_left_wheel" />
     <axis xyz="0 0 1" />
     <dynamics damping="0.2" />
   </joint>
-  <link name="front_left_wheel">
+  <link name="${prefix}front_left_wheel">
     <collision>
+      <!-- <origin xyz="0 0 .06" rpy="0 0 0" /> -->
       <origin xyz="0 0 .025" rpy="0 0 0" />
       <geometry>
@@ -57,6 +61,8 @@
     </collision>
     <visual>
+      <!-- <origin xyz="0 0 .06" rpy="0 0 0" /> -->
       <origin xyz="0 0 .025" rpy="0 0 0" />
       <geometry>
+        <!-- <sphere radius="0.3" /> -->
         <cylinder radius="0.05" length="0.05" />
       </geometry>
@@ -64,4 +70,5 @@
     </visual>
     <inertial>
+      <!-- <origin xyz="0 0 .06" rpy="0 0 0" /> -->
        <origin xyz="0 0 .025" rpy="0 0 0" />
       <mass value="0.5" />
@@ -74,13 +81,15 @@
     </inertial>
   </link>
-  <joint name="front_right_wheel_joint" type="continuous">
+  <!-- front right wheel -->
+  <joint name="${prefix}front_right_wheel_joint" type="continuous">
     <origin xyz="0.14 -0.15 0." rpy="-${pi/2} 0 0" />
-    <parent link="base_link" />
-    <child link="front_right_wheel" />
+    <parent link="${prefix}base_link" />
+    <child link="${prefix}front_right_wheel" />
     <axis xyz="0 0 1" />
     <dynamics damping="0.2" />
   </joint>
-  <link name="front_right_wheel">
+  <link name="${prefix}front_right_wheel">
     <collision>
+      <!-- <origin xyz="0 0 -.06" rpy="0 0 0" /> -->
       <origin xyz="0 0 -.025" rpy="0 0 0" />
       <geometry>
@@ -96,4 +105,5 @@
     </visual>
     <inertial>
+      <!-- <origin xyz="0 0 -.06" rpy="0 0 0" /> -->
       <origin xyz="0 0 -.025" rpy="0 0 0" />
       <mass value=".5" />
@@ -106,13 +116,15 @@
     </inertial>
   </link>
-  <joint name="rear_left_wheel_joint" type="continuous">
+  <!-- rear left wheel -->
+  <joint name="${prefix}rear_left_wheel_joint" type="continuous">
     <origin xyz="-0.14 0.15 0." rpy="-${pi/2} 0 0" />
-    <parent link="base_link" />
-    <child link="rear_left_wheel" />
+    <parent link="${prefix}base_link" />
+    <child link="${prefix}rear_left_wheel" />
     <axis xyz="0 0 1" />
     <dynamics damping="0.2" />
   </joint>
-  <link name="rear_left_wheel">
+  <link name="${prefix}rear_left_wheel">
     <collision>
+      <!-- <origin xyz="0 0 .06" rpy="0 0 0" /> -->
        <origin xyz="0 0 .025" rpy="0 0 0" />
       <geometry>
@@ -121,4 +133,5 @@
     </collision>
     <visual>
+      <!-- <origin xyz="0 0 .06" rpy="0 0 0" /> -->
        <origin xyz="0 0 .025" rpy="0 0 0" />
       <geometry>
@@ -128,4 +141,5 @@
     </visual>
     <inertial>
+      <!-- <origin xyz="0 0 .06" rpy="0 0 0" /> -->
        <origin xyz="0 0 .025" rpy="0 0 0" />
       <mass value="0.5" />
@@ -138,13 +152,15 @@
     </inertial>
   </link>
-  <joint name="rear_right_wheel_joint" type="continuous">
+  <!-- rear right wheel -->
+  <joint name="${prefix}rear_right_wheel_joint" type="continuous">
     <origin xyz="-0.14 -0.15 0." rpy="-${pi/2} 0 0" />
-    <parent link="base_link" />
-    <child link="rear_right_wheel" />
+    <parent link="${prefix}base_link" />
+    <child link="${prefix}rear_right_wheel" />
     <axis xyz="0 0 1" />
     <dynamics damping="0.2" />
   </joint>
-  <link name="rear_right_wheel">
+  <link name="${prefix}rear_right_wheel">
     <collision>
+      <!-- <origin xyz="0 0 -.06" rpy="0 0 0" /> -->
        <origin xyz="0 0 -.025" rpy="0 0 0" />
       <geometry>
@@ -153,4 +169,5 @@
     </collision>
     <visual>
+      <!-- <origin xyz="0 0 -.06" rpy="0 0 0" /> -->
        <origin xyz="0 0 -.025" rpy="0 0 0" />
       <geometry>
@@ -160,4 +177,5 @@
     </visual>
     <inertial>
+      <!-- <origin xyz="0 0 -.06" rpy="0 0 0" /> -->
        <origin xyz="0 0 -.025" rpy="0 0 0" />
       <mass value="0.5" />
@@ -170,3 +188,4 @@
     </inertial>
   </link>
+  </xacro:macro>
 </robot>

File: src/rmitbot_description/urdf/rmitbot_ros2_control.xacro (robot description, xacro)
@@ -1,4 +1,5 @@
 <?xml version="1.0"?>
 <robot name="rmitbot" xmlns:xacro="http://www.ros.org/wiki/xacro" >
+    <xacro:macro name="rmitbot_ros2_control" params="prefix">
     <ros2_control name="RobotSystem" type="system">
         <xacro:if value="$(arg use_sim)">
@@ -14,5 +15,5 @@
             </hardware>
         </xacro:unless>
-        <joint name="front_left_wheel_joint">
+        <joint name="${prefix}front_left_wheel_joint">
             <command_interface name="velocity">
                 <param name="min">-1</param>
@@ -22,5 +23,5 @@
             <state_interface name="velocity" />
         </joint>
-        <joint name="front_right_wheel_joint">
+        <joint name="${prefix}front_right_wheel_joint">
             <command_interface name="velocity">
                 <param name="min">-1</param>
@@ -30,5 +31,5 @@
             <state_interface name="velocity" />
         </joint>
-        <joint name="rear_left_wheel_joint">
+        <joint name="${prefix}rear_left_wheel_joint">
             <command_interface name="velocity">
                 <param name="min">-1</param>
@@ -38,5 +39,5 @@
             <state_interface name="velocity" />
         </joint>
-        <joint name="rear_right_wheel_joint">
+        <joint name="${prefix}rear_right_wheel_joint">
             <command_interface name="velocity">
                 <param name="min">-1</param>
@@ -46,5 +47,5 @@
             <state_interface name="velocity" />
         </joint>
-        <sensor name="imu_sensor">
+        <sensor name="${prefix}imu_sensor">
             <state_interface name="orientation.x" />
             <state_interface name="orientation.y" />
@@ -63,7 +64,9 @@
             <parameters>$(find rmitbot_controller)/config/rmitbot_controller.yaml</parameters>
             <ros>
-                <remapping>/mecanum_drive_controller/odom:=/odom</remapping>
+                <namespace>${prefix[:-1]}</namespace>
+                <remapping>diff_drive_controller/odom:=/${prefix}odom</remapping>
             </ros>
         </plugin>
     </gazebo>
+    </xacro:macro>
 </robot>
