Commit message: weird code

File: src/rmitbot_description/urdf/rmitbot.urdf.xacro (robot description, xacro)
@@ -4,4 +4,6 @@
     <xacro:arg name="use_sim" default="false"/>
     <xacro:arg name="use_mock_hardware" default="false"/>
+    <xacro:arg name="prefix" default=""/>
+    <xacro:property name="prefix" value="$(arg prefix)"/>
     <xacro:include filename="$(find rmitbot_description)/urdf/rmitbot_platform.xacro" />
     <xacro:include filename="$(find rmitbot_description)/urdf/rmitbot_gazebo.xacro" />
@@ -9,29 +11,35 @@
     <xacro:include filename="$(find rmitbot_description)/urdf/rmitbot_imu.xacro" />
     <xacro:include filename="$(find rmitbot_description)/urdf/rmitbot_laser.xacro" />
+    <!-- Instantiate the macros -->
+    <xacro:rmitbot_platform prefix="${prefix}"/>
+    <xacro:rmitbot_gazebo prefix="${prefix}"/>
+    <xacro:rmitbot_ros2_control prefix="${prefix}"/>
+    <xacro:rmitbot_imu prefix="${prefix}"/>
+    <!-- <xacro:rmitbot_laser prefix="${prefix}"/> -->
     <!-- Include the cliff sensor macro -->
-    <xacro:include filename="$(find rmitbot_cliff_sensor)/urdf/cliff_sensor.xacro" />
+    <!-- <xacro:include filename="$(find rmitbot_cliff_sensor)/urdf/cliff_sensor.xacro" /> -->
     <!-- Cliff Sensor 0 (Front Center) -->
-    <xacro:cliff_sensor name="cliff_sensor_0" parent="base_link">
+    <!-- <xacro:cliff_sensor name="${prefix}cliff_sensor_0" parent="${prefix}base_link">
         <origin xyz="0.2 0.0 0.11" rpy="0 1.5708 0" />
-    </xacro:cliff_sensor>
+    </xacro:cliff_sensor> -->
     <!-- Cliff Sensor 1 (Front Right) -->
-    <xacro:cliff_sensor name="cliff_sensor_1" parent="base_link">
+    <!-- <xacro:cliff_sensor name="${prefix}cliff_sensor_1" parent="${prefix}base_link">
         <origin xyz="0.16 -0.24 0.11" rpy="0 1.5708 0" />
-    </xacro:cliff_sensor>
+    </xacro:cliff_sensor> -->
     <!-- Cliff Sensor 2 (Back Right) -->
-    <xacro:cliff_sensor name="cliff_sensor_2" parent="base_link">
+    <!-- <xacro:cliff_sensor name="${prefix}cliff_sensor_2" parent="${prefix}base_link">
         <origin xyz="-0.16 -0.24 0.11" rpy="0 1.5708 0" />
-    </xacro:cliff_sensor>
+    </xacro:cliff_sensor> -->
     <!-- Cliff Sensor 3 (Back Center) -->
-    <xacro:cliff_sensor name="cliff_sensor_3" parent="base_link">
+    <!-- <xacro:cliff_sensor name="${prefix}cliff_sensor_3" parent="${prefix}base_link">
         <origin xyz="-0.2 0.0 0.11" rpy="0 1.5708 0" />
-    </xacro:cliff_sensor>
+    </xacro:cliff_sensor> -->
     <!-- Cliff Sensor 4 (Back Left) -->
-    <xacro:cliff_sensor name="cliff_sensor_4" parent="base_link">
+    <!-- <xacro:cliff_sensor name="${prefix}cliff_sensor_4" parent="${prefix}base_link">
         <origin xyz="-0.16 0.24 0.11" rpy="0 1.5708 0" />
-    </xacro:cliff_sensor>
+    </xacro:cliff_sensor> -->
     <!-- Cliff Sensor 5 (Front Left) -->
-    <xacro:cliff_sensor name="cliff_sensor_5" parent="base_link">
+    <!-- <xacro:cliff_sensor name="${prefix}cliff_sensor_5" parent="${prefix}base_link">
         <origin xyz="0.16 0.24 0.11" rpy="0 1.5708 0" />
-    </xacro:cliff_sensor>
+    </xacro:cliff_sensor> -->
 </robot>

File: src/rmitbot_description/urdf/rmitbot_gazebo.xacro (robot description, xacro)
@@ -2,8 +2,9 @@
 <!-- Gazebo file contains information regarding the lnks's physics (e.g., friction, stiffness, damping) -->
 <robot name="rmitbot" xmlns:xacro="http://ros.org/wiki/xacro" xmlns:gz="http://gazebosim.org/schema">
+<xacro:macro name="rmitbot_gazebo" params="prefix">
   <!-- Wheels -->
      <!-- To emulate Mecanum wheels in Gazebo with spherical collisions it
   requires a custom friction model so the vehicle can strafe left to right -->
-  <gazebo reference='front_left_wheel'>
+  <gazebo reference='${prefix}front_left_wheel'>
     <collision>
       <surface>
@@ -13,5 +14,5 @@
             <mu2>0.0</mu2>
             <!-- <fdir1 gz:expressed_in="base_link">1 -1 0</fdir1> -->
-            <fdir1 gz:expressed_in="base_footprint">1 -1 0</fdir1>
+            <fdir1 gz:expressed_in="${prefix}base_footprint">1 -1 0</fdir1>
           </ode>
         </friction>
@@ -19,5 +20,5 @@
     </collision>
   </gazebo>
-  <gazebo reference='front_right_wheel'>
+  <gazebo reference='${prefix}front_right_wheel'>
     <collision>
       <surface>
@@ -27,5 +28,5 @@
             <mu2>0.0</mu2>
             <!-- <fdir1 gz:expressed_in="base_link">1 1 0</fdir1> -->
-            <fdir1 gz:expressed_in="base_footprint">1 1 0</fdir1>
+            <fdir1 gz:expressed_in="${prefix}base_footprint">1 1 0</fdir1>
           </ode>
         </friction>
@@ -33,5 +34,5 @@
     </collision>
   </gazebo>
-  <gazebo reference='rear_left_wheel'>
+  <gazebo reference='${prefix}rear_left_wheel'>
     <collision>
       <surface>
@@ -41,5 +42,5 @@
             <mu2>0.0</mu2>
             <!-- <fdir1 gz:expressed_in="base_link">1 1 0</fdir1> -->
-            <fdir1 gz:expressed_in="base_footprint">1 1 0</fdir1>
+            <fdir1 gz:expressed_in="${prefix}base_footprint">1 1 0</fdir1>
           </ode>
         </friction>
@@ -47,5 +48,5 @@
     </collision>
   </gazebo>
-  <gazebo reference='rear_right_wheel'>
+  <gazebo reference='${prefix}rear_right_wheel'>
     <collision>
       <surface>
@@ -55,5 +56,5 @@
             <mu2>0.0</mu2>
             <!-- <fdir1 gz:expressed_in="base_link">1 -1 0</fdir1> -->
-            <fdir1 gz:expressed_in="base_footprint">1 -1 0</fdir1>
+            <fdir1 gz:expressed_in="${prefix}base_footprint">1 -1 0</fdir1>
           </ode>
         </friction>
@@ -61,3 +62,4 @@
     </collision>
   </gazebo>
+</xacro:macro>
 </robot>

File: src/rmitbot_description/urdf/rmitbot_imu.xacro (robot description, xacro)
@@ -1,5 +1,6 @@
 <?xml version="1.0"?>
 <robot xmlns:xacro="http://www.ros.org/wiki/xacro" name="rmitbot">
-    <link name="imu_link">
+<xacro:macro name="rmitbot_imu" params="prefix">
+    <link name="${prefix}imu_link">
         <inertial>
             <origin xyz="-0.0055 0.00017 0.00051" rpy="0 0 0" />
@@ -24,8 +25,8 @@
         </collision>
     </link>
-    <joint name="imu_joint" type="fixed">
+    <joint name="${prefix}imu_joint" type="fixed">
         <origin xyz="0 0 0.1" rpy="0 0 0" />
-        <parent link="base_link" />
-        <child link="imu_link" />
+        <parent link="${prefix}base_link" />
+        <child link="${prefix}imu_link" />
         <axis xyz="0 0 0" />
     </joint>
@@ -36,10 +37,10 @@
     </gazebo>
     <!-- Gazebo parameters for IMU, with noise-->
-  <gazebo reference="imu_link">
-    <sensor name="imu" type="imu">
+  <gazebo reference="${prefix}imu_link">
+    <sensor name="${prefix}imu" type="imu">
       <always_on>true</always_on>
       <update_rate>100</update_rate>
-      <gz_frame_id>imu_link</gz_frame_id>
-      <topic>imu</topic>
+      <gz_frame_id>${prefix}imu_link</gz_frame_id>
+      <topic>${prefix[:-1]}_imu</topic>
       <imu>
         <angular_velocity>
@@ -86,3 +87,4 @@
     </sensor>
   </gazebo>
+</xacro:macro>
 </robot>

File: src/rmitbot_description/urdf/rmitbot_laser.xacro (robot description, xacro)
@@ -1,5 +1,6 @@
 <?xml version="1.0"?>
 <robot xmlns:xacro="http://www.ros.org/wiki/xacro" name="rmitbot">
-    <link name="laser_link">
+<xacro:macro name="rmitbot_laser" params="prefix">
+    <link name="${prefix}laser_link">
         <inertial>
             <origin xyz="-0.012 -0.00038 -0.017" rpy="0 0 0" />
@@ -21,13 +22,13 @@
         </collision>
     </link>
-    <joint name="laser_joint" type="fixed">
+    <joint name="${prefix}laser_joint" type="fixed">
         <!-- <origin xyz="0. 0. 0.12" rpy="0 0 3.14" /> -->
         <origin xyz="0. 0. 0.12" rpy="0 0 0" />
-        <parent link="base_link" />
-        <child link="laser_link" />
+        <parent link="${prefix}base_link" />
+        <child link="${prefix}laser_link" />
         <axis xyz="0 0 0" />
     </joint>
-    <gazebo reference="laser_link">
-        <sensor name="lidar" type="gpu_lidar">
+    <gazebo reference="${prefix}laser_link">
+        <sensor name="${prefix}lidar" type="gpu_lidar">
             <plugin filename="gz-sim-sensors-system" name="gz::sim::systems::Sensors">
                 <render_engine>ogre</render_engine>
@@ -35,7 +36,7 @@
             <always_on>true</always_on>
             <visualize>true</visualize>
-            <topic>scan</topic>
+            <topic>${prefix[:-1]}_scan</topic>
             <update_rate>5</update_rate>
-            <gz_frame_id>laser_link</gz_frame_id>
+            <gz_frame_id>${prefix}laser_link</gz_frame_id>
             <lidar>
                 <scan>
@@ -65,3 +66,4 @@
         </sensor>
     </gazebo>
+</xacro:macro>
 </robot>

File: src/rmitbot_description/urdf/rmitbot_platform.xacro (robot description, xacro)
@@ -1,4 +1,5 @@
 <?xml version="1.0"?>
 <robot name="rmitbot" xmlns:xacro="http://www.ros.org/wiki/xacro" xmlns:gz="http://gazebosim.org/schema">
+<xacro:macro name="rmitbot_platform" params="prefix">
   <material name="orange">
     <color rgba="0.8 0.4 0.0 1.0" />
@@ -10,11 +11,11 @@
     <color rgba="1 1 1 1.0" />
   </material>
-  <link name="base_footprint" />
-  <joint name="base_joint" type="fixed">
-    <parent link="base_footprint" />
-    <child link="base_link" />
+  <link name="${prefix}base_footprint" />
+  <joint name="${prefix}base_joint" type="fixed">
+    <parent link="${prefix}base_footprint" />
+    <child link="${prefix}base_link" />
     <origin xyz="0 0 0.05" rpy="0 0 0" />
   </joint>
-  <link name="base_link">
+  <link name="${prefix}base_link">
     <collision>
       <origin xyz="0 0 0.05" rpy="0 0 0" />
@@ -42,12 +43,12 @@
     </inertial>
   </link>
-  <joint name="front_left_wheel_joint" type="continuous">
+  <joint name="${prefix}front_left_wheel_joint" type="continuous">
     <origin xyz="0.14 0.15 0" rpy="-${pi/2} 0 0" />
-    <parent link="base_link" />
-    <child link="front_left_wheel" />
+    <parent link="${prefix}base_link" />
+    <child link="${prefix}front_left_wheel" />
     <axis xyz="0 0 1" />
     <dynamics damping="0.2" />
   </joint>
-  <link name="front_left_wheel">
+  <link name="${prefix}front_left_wheel">
     <collision>
       <origin xyz="0 0 .025" rpy="0 0 0" />
@@ -74,12 +75,12 @@
     </inertial>
   </link>
-  <joint name="front_right_wheel_joint" type="continuous">
+  <joint name="${prefix}front_right_wheel_joint" type="continuous">
     <origin xyz="0.14 -0.15 0." rpy="-${pi/2} 0 0" />
-    <parent link="base_link" />
-    <child link="front_right_wheel" />
+    <parent link="${prefix}base_link" />
+    <child link="${prefix}front_right_wheel" />
     <axis xyz="0 0 1" />
     <dynamics damping="0.2" />
   </joint>
-  <link name="front_right_wheel">
+  <link name="${prefix}front_right_wheel">
     <collision>
       <origin xyz="0 0 -.025" rpy="0 0 0" />
@@ -106,12 +107,12 @@
     </inertial>
   </link>
-  <joint name="rear_left_wheel_joint" type="continuous">
+  <joint name="${prefix}rear_left_wheel_joint" type="continuous">
     <origin xyz="-0.14 0.15 0." rpy="-${pi/2} 0 0" />
-    <parent link="base_link" />
-    <child link="rear_left_wheel" />
+    <parent link="${prefix}base_link" />
+    <child link="${prefix}rear_left_wheel" />
     <axis xyz="0 0 1" />
     <dynamics damping="0.2" />
   </joint>
-  <link name="rear_left_wheel">
+  <link name="${prefix}rear_left_wheel">
     <collision>
        <origin xyz="0 0 .025" rpy="0 0 0" />
@@ -138,12 +139,12 @@
     </inertial>
   </link>
-  <joint name="rear_right_wheel_joint" type="continuous">
+  <joint name="${prefix}rear_right_wheel_joint" type="continuous">
     <origin xyz="-0.14 -0.15 0." rpy="-${pi/2} 0 0" />
-    <parent link="base_link" />
-    <child link="rear_right_wheel" />
+    <parent link="${prefix}base_link" />
+    <child link="${prefix}rear_right_wheel" />
     <axis xyz="0 0 1" />
     <dynamics damping="0.2" />
   </joint>
-  <link name="rear_right_wheel">
+  <link name="${prefix}rear_right_wheel">
     <collision>
        <origin xyz="0 0 -.025" rpy="0 0 0" />
@@ -170,3 +171,4 @@
     </inertial>
   </link>
+</xacro:macro>
 </robot>

File: src/rmitbot_description/urdf/rmitbot_ros2_control.xacro (robot description, xacro)
@@ -1,4 +1,5 @@
 <?xml version="1.0"?>
 <robot name="rmitbot" xmlns:xacro="http://www.ros.org/wiki/xacro" >
+<xacro:macro name="rmitbot_ros2_control" params="prefix">
     <ros2_control name="RobotSystem" type="system">
         <xacro:if value="$(arg use_sim)">
@@ -20,5 +21,5 @@
             </xacro:unless>
         </xacro:unless>
-        <joint name="front_left_wheel_joint">
+        <joint name="${prefix}front_left_wheel_joint">
             <command_interface name="velocity">
                 <param name="min">-1</param>
@@ -28,5 +29,5 @@
             <state_interface name="velocity" />
         </joint>
-        <joint name="front_right_wheel_joint">
+        <joint name="${prefix}front_right_wheel_joint">
             <command_interface name="velocity">
                 <param name="min">-1</param>
@@ -36,5 +37,5 @@
             <state_interface name="velocity" />
         </joint>
-        <joint name="rear_left_wheel_joint">
+        <joint name="${prefix}rear_left_wheel_joint">
             <command_interface name="velocity">
                 <param name="min">-1</param>
@@ -44,5 +45,5 @@
             <state_interface name="velocity" />
         </joint>
-        <joint name="rear_right_wheel_joint">
+        <joint name="${prefix}rear_right_wheel_joint">
             <command_interface name="velocity">
                 <param name="min">-1</param>
@@ -73,3 +74,4 @@
         </plugin>
     </gazebo>
+</xacro:macro>
 </robot>

Commit message: qol and camera

File: src/rmitbot_description/urdf/rmitbot.urdf.xacro (robot description, xacro)
@@ -10,27 +10,27 @@
     <!-- Include the cliff sensor macro -->
     <xacro:include filename="$(find rmitbot_cliff_sensor)/urdf/cliff_sensor.xacro" />
-    <!-- Cliff Sensor 0 (Front Center) -->
+    <!-- Cliff Sensor 0 (Front Left) -->
     <xacro:cliff_sensor name="cliff_sensor_0" parent="base_link">
-        <origin xyz="0.2 0.0 0.11" rpy="0 1.5708 0" />
+        <origin xyz="0.2 0.085 0.25" rpy="0 0.5236 0.2618" />
     </xacro:cliff_sensor>
-    <!-- Cliff Sensor 1 (Front Right) -->
+    <!-- Cliff Sensor 1 (Back Right) -->
     <xacro:cliff_sensor name="cliff_sensor_1" parent="base_link">
-        <origin xyz="0.16 -0.24 0.11" rpy="0 1.5708 0" />
+        <origin xyz="-0.2 -0.085 0.25" rpy="0 0.5236 -2.8798" />
     </xacro:cliff_sensor>
-    <!-- Cliff Sensor 2 (Back Right) -->
+    <!-- Cliff Sensor 2 (Faulty - Unused) -->
     <xacro:cliff_sensor name="cliff_sensor_2" parent="base_link">
-        <origin xyz="-0.16 -0.24 0.11" rpy="0 1.5708 0" />
+        <origin xyz="-0.16 -0.24 0.25" rpy="0 1.5708 0" />
     </xacro:cliff_sensor>
-    <!-- Cliff Sensor 3 (Back Center) -->
+    <!-- Cliff Sensor 3 (Front Center) -->
     <xacro:cliff_sensor name="cliff_sensor_3" parent="base_link">
-        <origin xyz="-0.2 0.0 0.11" rpy="0 1.5708 0" />
+        <origin xyz="0.2 0.0 0.25" rpy="0 0.5236 0" />
     </xacro:cliff_sensor>
-    <!-- Cliff Sensor 4 (Back Left) -->
+    <!-- Cliff Sensor 4 (Front Right) -->
     <xacro:cliff_sensor name="cliff_sensor_4" parent="base_link">
-        <origin xyz="-0.16 0.24 0.11" rpy="0 1.5708 0" />
+        <origin xyz="0.2 -0.085 0.25" rpy="0 0.5236 -0.2618" />
     </xacro:cliff_sensor>
-    <!-- Cliff Sensor 5 (Front Left) -->
+    <!-- Cliff Sensor 5 (Back Left) -->
     <xacro:cliff_sensor name="cliff_sensor_5" parent="base_link">
-        <origin xyz="0.16 0.24 0.11" rpy="0 1.5708 0" />
+        <origin xyz="-0.2 0.085 0.25" rpy="0 0.5236 2.8798" />
     </xacro:cliff_sensor>
 </robot>

File: src/rmitbot_description/urdf/rmitbot_ros2_control.xacro (robot description, xacro)
@@ -11,5 +11,5 @@
                 <plugin>rmitbot_firmware/RmitbotInterface</plugin>
                 <!-- <param name="port">/dev/esp32</param> -->
-                <param name="port">/dev/ttyUSB0</param>
+                <param name="port">/dev/ttyUSB1</param>
             </hardware>
         </xacro:unless>
