Commit message: pc

File: src/rmitbot_description/urdf/rmitbot.urdf.xacro (robot description, xacro)
@@ -1,6 +1,6 @@
 <?xml version="1.0"?>
-<robot name="rmitbot"
-    xmlns:xacro="http://ros.org/wiki/xacro">
-    <xacro:arg name="use_sim" default="false"/>
+<robot name="rmitbot" xmlns:xacro="http://ros.org/wiki/xacro">
+    <xacro:arg name="prefix" default=""/>
+    <xacro:arg name="has_cliff_sensor" default="true"/>
     <xacro:include filename="$(find rmitbot_description)/urdf/rmitbot_platform.xacro" />
     <xacro:include filename="$(find rmitbot_description)/urdf/rmitbot_gazebo.xacro" />
@@ -8,29 +8,36 @@
     <xacro:include filename="$(find rmitbot_description)/urdf/rmitbot_imu.xacro" />
     <xacro:include filename="$(find rmitbot_description)/urdf/rmitbot_laser.xacro" />
-    <!-- Include the cliff sensor macro -->
-    <xacro:include filename="$(find rmitbot_cliff_sensor)/urdf/cliff_sensor.xacro" />
-    <!-- Cliff Sensor 0 (Front Left) -->
-    <xacro:cliff_sensor name="cliff_sensor_0" parent="base_link">
-        <origin xyz="0.2 0.085 0.25" rpy="0 0.5236 0.2618" />
-    </xacro:cliff_sensor>
-    <!-- Cliff Sensor 1 (Back Right) -->
-    <xacro:cliff_sensor name="cliff_sensor_1" parent="base_link">
-        <origin xyz="-0.2 -0.085 0.25" rpy="0 0.5236 -2.8798" />
-    </xacro:cliff_sensor>
-    <!-- Cliff Sensor 2 (Faulty - Unused) -->
-    <xacro:cliff_sensor name="cliff_sensor_2" parent="base_link">
-        <origin xyz="-0.16 -0.24 0.25" rpy="0 1.5708 0" />
-    </xacro:cliff_sensor>
-    <!-- Cliff Sensor 3 (Front Center) -->
-    <xacro:cliff_sensor name="cliff_sensor_3" parent="base_link">
-        <origin xyz="0.2 0.0 0.25" rpy="0 0.5236 0" />
-    </xacro:cliff_sensor>
-    <!-- Cliff Sensor 4 (Front Right) -->
-    <xacro:cliff_sensor name="cliff_sensor_4" parent="base_link">
-        <origin xyz="0.2 -0.085 0.25" rpy="0 0.5236 -0.2618" />
-    </xacro:cliff_sensor>
-    <!-- Cliff Sensor 5 (Back Left) -->
-    <xacro:cliff_sensor name="cliff_sensor_5" parent="base_link">
-        <origin xyz="-0.2 0.085 0.25" rpy="0 0.5236 2.8798" />
-    </xacro:cliff_sensor>
+    <xacro:rmitbot_platform prefix="$(arg prefix)"/>
+    <xacro:rmitbot_gazebo prefix="$(arg prefix)"/>
+    <xacro:rmitbot_ros2_control prefix="$(arg prefix)"/>
+    <xacro:rmitbot_imu prefix="$(arg prefix)"/>
+    <xacro:rmitbot_laser prefix="$(arg prefix)"/>
+    <xacro:if value="$(arg has_cliff_sensor)">
+        <!-- Include the cliff sensor macro -->
+        <xacro:include filename="$(find rmitbot_cliff_sensor)/urdf/cliff_sensor.xacro" />
+        <!-- Cliff Sensor 0 (Front Left) -->
+        <xacro:cliff_sensor name="$(arg prefix)cliff_sensor_0" parent="$(arg prefix)base_link">
+            <origin xyz="0.2 0.085 0.25" rpy="0 0.5236 0.2618" />
+        </xacro:cliff_sensor>
+        <!-- Cliff Sensor 1 (Back Right) -->
+        <xacro:cliff_sensor name="$(arg prefix)cliff_sensor_1" parent="$(arg prefix)base_link">
+            <origin xyz="-0.2 -0.085 0.25" rpy="0 0.5236 -2.8798" />
+        </xacro:cliff_sensor>
+        <!-- Cliff Sensor 2 (Faulty - Unused) -->
+        <xacro:cliff_sensor name="$(arg prefix)cliff_sensor_2" parent="$(arg prefix)base_link">
+            <origin xyz="-0.16 -0.24 0.25" rpy="0 1.5708 0" />
+        </xacro:cliff_sensor>
+        <!-- Cliff Sensor 3 (Front Center) -->
+        <xacro:cliff_sensor name="$(arg prefix)cliff_sensor_3" parent="$(arg prefix)base_link">
+            <origin xyz="0.2 0.0 0.25" rpy="0 0.5236 0" />
+        </xacro:cliff_sensor>
+        <!-- Cliff Sensor 4 (Front Right) -->
+        <xacro:cliff_sensor name="$(arg prefix)cliff_sensor_4" parent="$(arg prefix)base_link">
+            <origin xyz="0.2 -0.085 0.25" rpy="0 0.5236 -0.2618" />
+        </xacro:cliff_sensor>
+        <!-- Cliff Sensor 5 (Back Left) -->
+        <xacro:cliff_sensor name="$(arg prefix)cliff_sensor_5" parent="$(arg prefix)base_link">
+            <origin xyz="-0.2 0.085 0.25" rpy="0 0.5236 2.8798" />
+        </xacro:cliff_sensor>
+    </xacro:if>
 </robot>

File: src/rmitbot_description/urdf/rmitbot_ros2_control.xacro (robot description, xacro)
@@ -1,18 +1,12 @@
 <?xml version="1.0"?>
-<robot name="rmitbot" xmlns:xacro="http://www.ros.org/wiki/xacro" >
-    <ros2_control name="RobotSystem" type="system">
-        <xacro:if value="$(arg use_sim)">
-            <hardware>
-                <plugin>gz_ros2_control/GazeboSimSystem</plugin>
-            </hardware>
-        </xacro:if>
-        <xacro:unless value="$(arg use_sim)">
-            <hardware>
-                <plugin>rmitbot_firmware/RmitbotInterface</plugin>
-                <!-- <param name="port">/dev/esp32</param> -->
-                <param name="port">/dev/ttyUSB0</param>
-            </hardware>
-        </xacro:unless>
-        <joint name="front_left_wheel_joint">
+<robot name="rmitbot" xmlns:xacro="http://www.ros.org/wiki/xacro">
+<!-- Define the vehicles hardware,
+    command and state interfaces  -->
+     <xacro:macro name="rmitbot_ros2_control" params="prefix">
+     <ros2_control name="GazeboSimSystem" type="system">
+        <hardware>
+            <plugin>gz_ros2_control/GazeboSimSystem</plugin>
+        </hardware>
+        <joint name="${prefix}front_left_wheel_joint">
             <command_interface name="velocity">
                 <param name="min">-1</param>
@@ -22,5 +16,5 @@
             <state_interface name="velocity" />
         </joint>
-        <joint name="front_right_wheel_joint">
+        <joint name="${prefix}front_right_wheel_joint">
             <command_interface name="velocity">
                 <param name="min">-1</param>
@@ -30,5 +24,5 @@
             <state_interface name="velocity" />
         </joint>
-        <joint name="rear_left_wheel_joint">
+        <joint name="${prefix}rear_left_wheel_joint">
             <command_interface name="velocity">
                 <param name="min">-1</param>
@@ -38,5 +32,5 @@
             <state_interface name="velocity" />
         </joint>
-        <joint name="rear_right_wheel_joint">
+        <joint name="${prefix}rear_right_wheel_joint">
             <command_interface name="velocity">
                 <param name="min">-1</param>
@@ -46,24 +40,15 @@
             <state_interface name="velocity" />
         </joint>
-        <sensor name="imu_sensor">
-            <state_interface name="orientation.x" />
-            <state_interface name="orientation.y" />
-            <state_interface name="orientation.z" />
-            <state_interface name="orientation.w" />
-            <state_interface name="angular_velocity.x" />
-            <state_interface name="angular_velocity.y" />
-            <state_interface name="angular_velocity.z" />
-            <state_interface name="linear_acceleration.x" />
-            <state_interface name="linear_acceleration.y" />
-            <state_interface name="linear_acceleration.z" />
-        </sensor>
     </ros2_control>
-    <gazebo>
+    <!-- ROS2 Control plugin and topic re-mapping -->
+  <gazebo>
         <plugin filename="gz_ros2_control-system" name="gz_ros2_control::GazeboSimROS2ControlPlugin">
             <parameters>$(find rmitbot_controller)/config/rmitbot_controller.yaml</parameters>
             <ros>
-                <remapping>/mecanum_drive_controller/odom:=/odom</remapping>
+                <namespace>${prefix[:-1]}</namespace>
+                <remapping>diff_drive_controller/odom:=/${prefix}odom</remapping>
             </ros>
         </plugin>
     </gazebo>
+     </xacro:macro>
 </robot>

Commit message: final debug

File: src/rmitbot_description/urdf/rmitbot.urdf.xacro (robot description, xacro)
@@ -10,25 +10,9 @@
     <!-- Include the cliff sensor macro -->
     <xacro:include filename="$(find rmitbot_cliff_sensor)/urdf/cliff_sensor.xacro" />
-    <!-- Cliff Sensor 0 (Front Left) -->
-    <xacro:cliff_sensor name="cliff_sensor_0" parent="base_link">
-        <origin xyz="0.2 0.085 0.25" rpy="0 0.5236 0.2618" />
-    </xacro:cliff_sensor>
-    <!-- Cliff Sensor 1 (Back Right) -->
-    <xacro:cliff_sensor name="cliff_sensor_1" parent="base_link">
-        <origin xyz="-0.2 -0.085 0.25" rpy="0 0.5236 -2.8798" />
-    </xacro:cliff_sensor>
-    <!-- Cliff Sensor 2 (Faulty - Unused) -->
-    <xacro:cliff_sensor name="cliff_sensor_2" parent="base_link">
-        <origin xyz="-0.16 -0.24 0.25" rpy="0 1.5708 0" />
-    </xacro:cliff_sensor>
     <!-- Cliff Sensor 3 (Front Center) -->
     <xacro:cliff_sensor name="cliff_sensor_3" parent="base_link">
         <origin xyz="0.2 0.0 0.25" rpy="0 0.5236 0" />
     </xacro:cliff_sensor>
-    <!-- Cliff Sensor 4 (Front Right) -->
-    <xacro:cliff_sensor name="cliff_sensor_4" parent="base_link">
-        <origin xyz="0.2 -0.085 0.25" rpy="0 0.5236 -0.2618" />
-    </xacro:cliff_sensor>
-    <!-- Cliff Sensor 5 (Back Left) -->
+    <!-- Cliff Sensor 5 (Back Left - Used as Back) -->
     <xacro:cliff_sensor name="cliff_sensor_5" parent="base_link">
         <origin xyz="-0.2 0.085 0.25" rpy="0 0.5236 2.8798" />

Commit message: cliff remove swarm

File: src/rmitbot_description/urdf/rmitbot.urdf.xacro (robot description, xacro)
@@ -8,13 +8,3 @@
     <xacro:include filename="$(find rmitbot_description)/urdf/rmitbot_imu.xacro" />
     <xacro:include filename="$(find rmitbot_description)/urdf/rmitbot_laser.xacro" />
-    <!-- Include the cliff sensor macro -->
-    <xacro:include filename="$(find rmitbot_cliff_sensor)/urdf/cliff_sensor.xacro" />
-    <!-- Cliff Sensor 3 (Front Center) -->
-    <xacro:cliff_sensor name="cliff_sensor_3" parent="base_link">
-        <origin xyz="0.2 0.0 0.25" rpy="0 0.5236 0" />
-    </xacro:cliff_sensor>
-    <!-- Cliff Sensor 5 (Back Left - Used as Back) -->
-    <xacro:cliff_sensor name="cliff_sensor_5" parent="base_link">
-        <origin xyz="-0.2 0.085 0.25" rpy="0 0.5236 2.8798" />
-    </xacro:cliff_sensor>
 </robot>
