Commit message: Parameterize URDF and Controller Configs for Small and Big Robots

File: src/rmitbot_description/urdf/bigbot.urdf.xacro (robot description, xacro)
@@ -1,11 +1,10 @@
 <?xml version="1.0"?>
-<robot name="rmitbot"
-    xmlns:xacro="http://ros.org/wiki/xacro">
+<robot name="rmitbot_big" xmlns:xacro="http://ros.org/wiki/xacro">
     <xacro:arg name="use_sim" default="false"/>
     <xacro:arg name="controller_serial_port" default="/dev/serial/by-id/usb-1a86_USB_Serial-if00-port0"/>
-    <xacro:property name="wheel_radius" value="0.13" />
-    <xacro:property name="wheel_track_y" value="0.36" />
-    <xacro:property name="wheel_base_x" value="0.19" />
-    <xacro:property name="lidar_z" value="0.27" />
+    <xacro:property name="wheel_radius" value="0.25" />
+    <xacro:property name="wheel_track_y" value="0.61" />
+    <xacro:property name="wheel_base_x" value="0.33" />
+    <xacro:property name="lidar_z" value="0.37" />
     <xacro:include filename="$(find rmitbot_description)/urdf/rmitbot_platform.xacro" />
     <xacro:include filename="$(find rmitbot_description)/urdf/rmitbot_gazebo.xacro" />

File: src/rmitbot_description/urdf/rmitbot_laser.xacro (robot description, xacro)
@@ -23,5 +23,5 @@
     <joint name="laser_joint" type="fixed">
         <!-- <origin xyz="0. 0. 0.12" rpy="0 0 3.14" /> -->
-        <origin xyz="0. 0. 0.12" rpy="0 0 0" />
+        <origin xyz="0. 0. ${lidar_z}" rpy="0 0 0" />
         <parent link="base_link" />
         <child link="laser_link" />

File: src/rmitbot_description/urdf/rmitbot_platform.xacro (robot description, xacro)
@@ -14,5 +14,5 @@
     <parent link="base_footprint" />
     <child link="base_link" />
-    <origin xyz="0 0 0.05" rpy="0 0 0" />
+    <origin xyz="0 0 ${wheel_radius}" rpy="0 0 0" />
   </joint>
   <link name="base_link">
@@ -20,5 +20,5 @@
       <origin xyz="0 0 0.05" rpy="0 0 0" />
       <geometry>
-         <box size=".28 .3 0.1" />
+         <box size="${wheel_base_x + 0.10} ${wheel_track_y - 0.05} 0.1" />
       </geometry>
     </collision>
@@ -26,5 +26,5 @@
       <origin xyz="0 0 0.05" rpy="0 0 0" />
       <geometry>
-         <box size=".28 .3 0.1" />
+         <box size="${wheel_base_x + 0.10} ${wheel_track_y - 0.05} 0.1" />
       </geometry>
       <material name="orange" />
@@ -43,5 +43,5 @@
   </link>
   <joint name="front_left_wheel_joint" type="continuous">
-    <origin xyz="0.14 0.15 0" rpy="-${pi/2} 0 0" />
+    <origin xyz="${wheel_base_x/2} ${wheel_track_y/2} 0" rpy="-${pi/2} 0 0" />
     <parent link="base_link" />
     <child link="front_left_wheel" />
@@ -53,5 +53,5 @@
       <origin xyz="0 0 .025" rpy="0 0 0" />
       <geometry>
-        <sphere radius="0.05" />
+        <sphere radius="${wheel_radius}" />
       </geometry>
     </collision>
@@ -59,5 +59,5 @@
       <origin xyz="0 0 .025" rpy="0 0 0" />
       <geometry>
-        <cylinder radius="0.05" length="0.05" />
+        <cylinder radius="${wheel_radius}" length="0.05" />
       </geometry>
       <material name="black" />
@@ -75,5 +75,5 @@
   </link>
   <joint name="front_right_wheel_joint" type="continuous">
-    <origin xyz="0.14 -0.15 0." rpy="-${pi/2} 0 0" />
+    <origin xyz="${wheel_base_x/2} -${wheel_track_y/2} 0." rpy="-${pi/2} 0 0" />
     <parent link="base_link" />
     <child link="front_right_wheel" />
@@ -85,5 +85,5 @@
       <origin xyz="0 0 -.025" rpy="0 0 0" />
       <geometry>
-        <sphere radius="0.05" />
+        <sphere radius="${wheel_radius}" />
       </geometry>
     </collision>
@@ -91,5 +91,5 @@
       <origin xyz="0 0 -.025" rpy="0 0 0" />
       <geometry>
-        <cylinder radius="0.05" length="0.05" />
+        <cylinder radius="${wheel_radius}" length="0.05" />
       </geometry>
       <material name="black" />
@@ -107,5 +107,5 @@
   </link>
   <joint name="rear_left_wheel_joint" type="continuous">
-    <origin xyz="-0.14 0.15 0." rpy="-${pi/2} 0 0" />
+    <origin xyz="-${wheel_base_x/2} ${wheel_track_y/2} 0." rpy="-${pi/2} 0 0" />
     <parent link="base_link" />
     <child link="rear_left_wheel" />
@@ -117,5 +117,5 @@
        <origin xyz="0 0 .025" rpy="0 0 0" />
       <geometry>
-        <sphere radius="0.05" />
+        <sphere radius="${wheel_radius}" />
       </geometry>
     </collision>
@@ -123,5 +123,5 @@
        <origin xyz="0 0 .025" rpy="0 0 0" />
       <geometry>
-        <cylinder radius="0.05" length="0.05" />
+        <cylinder radius="${wheel_radius}" length="0.05" />
       </geometry>
       <material name="black" />
@@ -139,5 +139,5 @@
   </link>
   <joint name="rear_right_wheel_joint" type="continuous">
-    <origin xyz="-0.14 -0.15 0." rpy="-${pi/2} 0 0" />
+    <origin xyz="-${wheel_base_x/2} -${wheel_track_y/2} 0." rpy="-${pi/2} 0 0" />
     <parent link="base_link" />
     <child link="rear_right_wheel" />
@@ -149,5 +149,5 @@
        <origin xyz="0 0 -.025" rpy="0 0 0" />
       <geometry>
-        <sphere radius="0.05" />
+        <sphere radius="${wheel_radius}" />
       </geometry>
     </collision>
@@ -155,5 +155,5 @@
        <origin xyz="0 0 -.025" rpy="0 0 0" />
       <geometry>
-        <cylinder radius="0.05" length="0.05" />
+        <cylinder radius="${wheel_radius}" length="0.05" />
       </geometry>
       <material name="black" />

File: src/rmitbot_description/urdf/smallbot.urdf.xacro (robot description, xacro)
@@ -1,5 +1,4 @@
 <?xml version="1.0"?>
-<robot name="rmitbot"
-    xmlns:xacro="http://ros.org/wiki/xacro">
+<robot name="rmitbot_small" xmlns:xacro="http://ros.org/wiki/xacro">
     <xacro:arg name="use_sim" default="false"/>
     <xacro:arg name="controller_serial_port" default="/dev/serial/by-id/usb-1a86_USB_Serial-if00-port0"/>

Commit message: Fix wheel radius from diameter and split joy_node to separate devices

File: src/rmitbot_description/urdf/bigbot.urdf.xacro (robot description, xacro)
@@ -3,5 +3,5 @@
     <xacro:arg name="use_sim" default="false"/>
     <xacro:arg name="controller_serial_port" default="/dev/serial/by-id/usb-1a86_USB_Serial-if00-port0"/>
-    <xacro:property name="wheel_radius" value="0.25" />
+    <xacro:property name="wheel_radius" value="0.125" />
     <xacro:property name="wheel_track_y" value="0.61" />
     <xacro:property name="wheel_base_x" value="0.33" />

File: src/rmitbot_description/urdf/rmitbot.urdf.xacro (robot description, xacro)
@@ -4,5 +4,5 @@
     <xacro:arg name="use_sim" default="false"/>
     <xacro:arg name="controller_serial_port" default="/dev/serial/by-id/usb-1a86_USB_Serial-if00-port0"/>
-    <xacro:property name="wheel_radius" value="0.13" />
+    <xacro:property name="wheel_radius" value="0.065" />
     <xacro:property name="wheel_track_y" value="0.36" />
     <xacro:property name="wheel_base_x" value="0.19" />

File: src/rmitbot_description/urdf/smallbot.urdf.xacro (robot description, xacro)
@@ -3,5 +3,5 @@
     <xacro:arg name="use_sim" default="false"/>
     <xacro:arg name="controller_serial_port" default="/dev/serial/by-id/usb-1a86_USB_Serial-if00-port0"/>
-    <xacro:property name="wheel_radius" value="0.13" />
+    <xacro:property name="wheel_radius" value="0.065" />
     <xacro:property name="wheel_track_y" value="0.36" />
     <xacro:property name="wheel_base_x" value="0.19" />

Commit message: Update bigbot wheelbase to 0.31

File: src/rmitbot_description/urdf/bigbot.urdf.xacro (robot description, xacro)
@@ -5,5 +5,5 @@
     <xacro:property name="wheel_radius" value="0.125" />
     <xacro:property name="wheel_track_y" value="0.61" />
-    <xacro:property name="wheel_base_x" value="0.33" />
+    <xacro:property name="wheel_base_x" value="0.31" />
     <xacro:property name="lidar_z" value="0.37" />
     <xacro:include filename="$(find rmitbot_description)/urdf/rmitbot_platform.xacro" />
